File: hardware/AR-Breakout/AR-Breakout.kicad_pcb (KiCad board)
At the start: 2 copper layers, 0 parts

Commit message: schem progress
Parts:
- added C1: .1uF, Capacitor_SMD:C_0805_2012Metric_Pad1.18x1.45mm_HandSolder, F.Cu at (127.4, 137.8)
- added C2: .1uF, Capacitor_SMD:C_0805_2012Metric_Pad1.18x1.45mm_HandSolder, F.Cu at (127.4, 140.8)
- added D2: LED, LED_SMD:LED_0805_2012Metric_Pad1.15x1.40mm_HandSolder, F.Cu at (154.7, 90.6)
- added D3: LED, LED_SMD:LED_0805_2012Metric_Pad1.15x1.40mm_HandSolder, F.Cu at (154.7, 93.7)
- added D4: LED, LED_SMD:LED_0805_2012Metric_Pad1.15x1.40mm_HandSolder, F.Cu at (154.7, 96.7)
- added D5: LED, LED_SMD:LED_0805_2012Metric_Pad1.15x1.40mm_HandSolder, F.Cu at (131.6, 125.7)
- added J3: Logic Analyzer, AR-footprints:CONN_SFH11-xxxC-D05-ST-XX_SUL, F.Cu at (123.6, 116.1)
- added JP1: SolderJumper_2_Open, Resistor_SMD:R_0805_2012Metric_Pad1.20x1.40mm_HandSolder, F.Cu at (149.9, 90.6)
- added R1: 1k, Resistor_SMD:R_0805_2012Metric_Pad1.20x1.40mm_HandSolder, F.Cu at (149.9, 93.5)
- added R2: 1k, Resistor_SMD:R_0805_2012Metric_Pad1.20x1.40mm_HandSolder, F.Cu at (149.9, 96.5)
- added R3: 1k, Resistor_SMD:R_0805_2012Metric_Pad1.20x1.40mm_HandSolder, F.Cu at (149.9, 99.4)
- added R4: 1k, Resistor_SMD:R_0805_2012Metric_Pad1.20x1.40mm_HandSolder, F.Cu at (131.6, 128.7)
- added R5: 1k, Resistor_SMD:R_0805_2012Metric_Pad1.20x1.40mm_HandSolder, F.Cu at (120.3, 133.8)
- added TP3: TestPoint, TestPoint:TestPoint_Pad_2.0x2.0mm, F.Cu at (119.3, 144.0)
- added TP4: TestPoint, TestPoint:TestPoint_Loop_D3.80mm_Drill2.0mm, F.Cu at (120.1, 139.1)
- added U1: SEEEDUINO-XIAO-ESP32C3, AR-footprints:MOUDLE14P-SMD-2.54-21X17.8MM, F.Cu at (116.6, 110.3)
- added U2: TXS0108EPWR, AR-footprints:TXS0108EPWR, F.Cu at (122.8, 128.3)
