File: hardware/AR-Breakout/AR-Breakout.kicad_sch (KiCad schematic)
At the start: 2 parts, among them J1 Barrel_Jack_MountingPin, J3 Logic Analyzer

Commit message: PCB
Parts:
- removed J1: Barrel_Jack_MountingPin, symbol Connector:Barrel_Jack_MountingPin
- added D3, D4: LED, LED_SMD:LED_0805_2012Metric_Pad1.15x1.40mm_HandSolder, symbol Device:LED
- added D6, D7, D8: PWR_LED, LED_SMD:LED_0805_2012Metric_Pad1.15x1.40mm_HandSolder, symbol Device:LED
- added H1, H2: MountingHole_Pad, MountingHole:MountingHole_2.5mm_Pad, symbol Mechanical:MountingHole_Pad
- added J1: 5V_Inject, Connector_PinHeader_2.54mm:PinHeader_1x02_P2.54mm_Vertical, symbol Connector_Generic:Conn_01x02
- added J4: 3.3V_Inject, Connector_PinHeader_2.54mm:PinHeader_1x02_P2.54mm_Vertical, symbol Connector_Generic:Conn_01x02
- added J5: Barrel_Jack_Switch, Connector_BarrelJack:BarrelJack_GCT_DCJ200-10-A_Horizontal, symbol Connector:Barrel_Jack_Switch
- added R10, R6, R7, R8, R9: 1k, Resistor_SMD:R_0805_2012Metric_Pad1.20x1.40mm_HandSolder, symbol Device:R
- added TP1, TP5, TP7, TP8: TestPoint, TestPoint:TestPoint_THTPad_D3.0mm_Drill1.5mm, symbol Connector:TestPoint
Connections:
- net +3.3V: now also J4.1 (Pin_1), R8.1, TP8.1
- net GND: now also D3.1 (K), D4.1 (K), D6.1 (K), D7.1 (K), D8.1 (K), J1.2 (Pin_2), J4.2 (Pin_2), J5.2, TP1.1
- net ultra96_pwrOut: now also J5.1, R6.1, TP5.1
- net extra_io_1: now reaches J3.4 (CH6)
- net extra_io_0: now reaches J3.6 (CH4)
- net uart0_rx: no longer names the net of J3.9 (CH1)
- net uart0_tx: no longer names the net of J3.7 (CH3)
- net uart1_rx renamed pl_breathe_out
- net pl_breathe_out: now also R9.1
- net uart1_tx renamed pl_breathe_in
- net pl_breathe_in: now also R10.1
- new net: D3.2 (A), R9.2
- new net: D8.2 (A), R8.2
- new net: D4.2 (A), R10.2
- new net: D6.2 (A), R6.2
- new net: D7.2 (A), R7.2
- new net +5V: J1.1 (Pin_1), R7.1, TP7.1
- no-connect marks 1 -> 7
Other:
- removed sheet esp32
- removed sheet imu
- added sheet 5-3.3V_LDO (5-3.3V_LDO.kicad_sch)
- sheet ultra96 ports: added extra_io_0, extra_io_1, pl_breathe_in, pl_breathe_out, ultra96_5V; removed {ultra96_uart0}, {ultra96_uart1}
- note added: "Power is coming from USB-C PD Trigger Board"
- note added: "To the Ultra96"
