File: hardware/AR-Breakout/UsbPowerDist.kicad_sch (KiCad schematic)
At the start: 0 parts

Commit message: PCB
Parts:
- added TP6: TestPoint, TestPoint:TestPoint_THTPad_D3.0mm_Drill1.5mm, symbol Connector:TestPoint
- added U3: ~, AR-footprints:USB-C-TRIGGER, symbol AR-symbols:USB_C_Trigger
Connections:
- net ultra96_pwrOut: now also U3.1 (+), U3.2 (+)
- new net GND: TP6.1, U3.3 (-), U3.4 (-)
