File: hardware/AR-Breakout/esp32.kicad_sch (KiCad schematic)
At the start: 13 parts, among them U1 SEEEDUINO-XIAO-ESP32C3

Commit message: PCB
Connections:
- net esp_3V3: no longer R1.1
- net esp_3v3: now also R1.1
Changed lines of the file:
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@@
 		)
 	)
-	(wire
-		(pts
-			(xy 223.52 76.2) (xy 231.14 76.2)
-		)
-		(stroke
-			(width 0)
-			(type default)
-		)
-	)
 	(image
 		(at 76.2 45.72)
@@
 		)
 	)
-	(label "esp_3V3"
-		(at 231.14 76.2 180)
-		(effects
-			(font
-				(size 1.27 1.27)
-			)
-			(justify right bottom)
-		)
-	)
 	(label "esp_connected"
 		(at 176.53 92.71 180)
@@
 		(effects
 			(font
+				(size 1.27 1.27)
+			)
+			(justify left)
+		)
+	)
+	(hierarchical_label "esp_3v3"
+		(shape input)
+		(at 223.52 76.2 0)
+		(effects
+			(font
