File: hardware/AR-Breakout/ultra96.kicad_sch (KiCad schematic)
At the start: 3 parts

Commit message: PCB
Parts:
- removed TP4: TestPoint, TestPoint:TestPoint_Loop_D3.80mm_Drill2.0mm, symbol Connector:TestPoint
- J2: footprint (none) -> AR-footprints:TW2002TD170SM
Connections:
- net pl_breathe_in_1v8: now reaches J2.3 (HD_GPIO_0)
- net extra_io_1_1v8: now reaches J2.9 (HD_GPIO_3)
- net pl_heartbeat: no longer names the net of J2.23 (MIO36_PS_GPIO1_0)
- net ultra96_5v renamed ultra96_5V
- net ultra96_uart0_rx renamed extra_io_0_1v8
- net ultra96_uart0_tx renamed pl_breathe_out_1v8
- net ultra96_uart1_rx: no longer names the net of J2.13 (HD_GPIO_5)
- net ultra96_uart1_tx: no longer names the net of J2.11 (HD_GPIO_4)
- no-connect marks 2 -> 76
Other:
- added sheet 1.8v_Led (1.8v_Led.kicad_sch)
- added sheet 1.8v_Led1 (1.8v_Led.kicad_sch)
